Commit message: Tuned PID, Added Camera and Lidar

File: revolt_description/urdf/include/revolt_control.xacro (robot description, xacro)
@@ -8,4 +8,5 @@
     <param name="left_wheel_name">left_wheel_joint</param>
     <param name="right_wheel_name">right_wheel_joint</param>
+    <param name="loop_rate">30</param>
     <param name="serial_device">/dev/ttyUSB_ARDUINO</param>
     <param name="baud_rate">57600</param>

File: revolt_description/urdf/revolt.urdf.xacro (robot description, xacro)
@@ -3,4 +3,5 @@
     <xacro:property name="package_name" value="revolt_description" />
     <xacro:property name="robot_name" value="revolt" />
+    <xacro:arg name="use_fixed_caster" default="True"/>
     <xacro:arg name="use_real_ros_control" default="True" />
     <!-- ................................ BASE LINK .................................. -->
@@ -108,5 +109,5 @@
         <parent link="base_link" />
         <child link="chassis" />
-        <origin xyz="0 0 0" rpy="0 0 0" />
+        <origin xyz="0 0 0" rpy="0 0 ${pi}" />
     </joint>
     <!-- ................................ IMU .................................. -->
@@ -268,5 +269,5 @@
         </inertial>
     </link>
-    <xacro:if value="$(arg use_real_ros_control)">
+    <xacro:if value="$(arg use_fixed_caster)">
         <joint name="frontcaster_wheel_joint" type="fixed">
             <origin xyz="0.013500000000000025868 3.1212253173671393473e-18 -0.017000000000000001221"
@@ -275,6 +276,4 @@
             <child link="caster_wheel" />
             <axis xyz="0 0 1" />
-            <limit effort="1" velocity="20" />
-            <joint_properties friction="0.0" />
         </joint>
         <joint name="frontcaster_rotation_joint" type="fixed">
@@ -285,9 +284,7 @@
             <child link="caster_punch_bracket" />
             <axis xyz="0 0 1" />
-            <limit effort="1" velocity="20" />
-            <joint_properties friction="0.0" />
         </joint>
     </xacro:if>
-    <xacro:unless value="$(arg use_real_ros_control)">
+    <xacro:unless value="$(arg use_fixed_caster)">
         <joint name="frontcaster_wheel_joint" type="continuous">
             <origin xyz="0.013500000000000025868 3.1212253173671393473e-18 -0.017000000000000001221"
@@ -353,5 +350,5 @@
         </inertial>
     </link>
-    <xacro:if value="$(arg use_real_ros_control)">
+    <xacro:if value="$(arg use_fixed_caster)">
         <joint name="backcaster_wheel_joint" type="fixed">
             <origin xyz="0.013499999999999998113 2.2538635793787358001e-18 -0.017000000000000001221"
@@ -360,6 +357,4 @@
             <child link="caster_wheel_2" />
             <axis xyz="0 0 1" />
-            <limit effort="1" velocity="20" />
-            <joint_properties friction="0.0" />
         </joint>
         <joint name="backcaster_rotation_joint" type="fixed">
@@ -370,9 +365,7 @@
             <child link="caster_punch_bracket_2" />
             <axis xyz="0 0 1" />
-            <limit effort="1" velocity="20" />
-            <joint_properties friction="0.0" />
         </joint>
     </xacro:if>
-    <xacro:unless value="$(arg use_real_ros_control)">
+    <xacro:unless value="$(arg use_fixed_caster)">
         <joint name="backcaster_wheel_joint" type="continuous">
             <origin xyz="0.013499999999999998113 2.2538635793787358001e-18 -0.017000000000000001221"
